Commit message: xArm integration

File: create_description/urdf/create_2.urdf.xacro (robot description, xacro)
@@ -3,6 +3,13 @@
   <xacro:include filename="$(find create_description)/urdf/create_base.urdf.xacro" />
   <xacro:include filename="$(find create_description)/urdf/create_2_gazebo.urdf.xacro" />
+  <xacro:include filename="$(find xarm_description)/urdf/xarm.urdf"/>
   <xacro:create_base wheel_separation="0.235" base_diameter="0.3485">
     <mesh filename="package://create_description/meshes/create_2.dae" />
   </xacro:create_base>
+  <xacro:property name="PI" value="3.1415926535897931" />
+  <joint name="xarm_base_joint" type="fixed">
+        <parent link="base_footprint"/>
+        <child link="xarm_base_link"/>
+        <origin xyz="0.095 0.0 0.175" rpy="0.0 0.0 ${PI/2}"/>
+  </joint>
 </robot>

File: create_description/urdf/create_base.urdf.xacro (robot description, xacro)
@@ -29,5 +29,6 @@
     </joint>
   </xacro:macro>
-  <xacro:macro name="create_base" params="diffdrive_update_rate:=40 wheel_separation wheel_radius:=0.036 wheel_width:=0.024 wheel_torque:=1.0 wheel_accel:=1.8 mass_kg:=3.5 base_diameter *mesh">
+  <!--xacro:macro name="create_base" params="diffdrive_update_rate:=40 wheel_separation wheel_radius:=0.036 wheel_width:=0.024 wheel_torque:=1.0 wheel_accel:=1.8 mass_kg:=3.5 base_diameter *mesh"-->
+  <xacro:macro name="create_base" params="diffdrive_update_rate:=40 wheel_separation wheel_radius:=0.01 wheel_width:=0.024 wheel_torque:=1.0 wheel_accel:=1.8 mass_kg:=3.5 base_diameter *mesh">
     <xacro:include filename="$(find create_description)/urdf/create_base_gazebo.urdf.xacro" />
     <link name="base_footprint">
@@ -49,5 +50,5 @@
     <inertial>
       <mass value="2" />
-      <origin xyz="0 0 0.0" />
+      <origin xyz="0 0 0" />
       <inertia ixx="0.01" ixy="0.0" ixz="0.0" iyy="0.01" iyz="0.0" izz="0.5" />
     </inertial>
@@ -123,8 +124,29 @@
         <origin xyz="0 0 0" rpy="0 0 0" />
         <geometry>
-          <box size="0.110 0.025 0.015" />
+          <box size="0.025 0.110 0.015" />
         </geometry>
         <material name="Black" />
       </visual>
+    </link>
+    <link name="vertical_body">
+      <inertial>
+        <mass value="0.01" />
+        <origin xyz="0.0 0.0 0.0"/>
+        <inertia ixx="0.001" ixy="0.0" ixz="0.0" iyy="0.001" iyz="0.0" izz="0.001" />
+      </inertial>
+      <visual>
+        <origin xyz="0 0 0.255" rpy="0 0 0" />
+        <geometry>
+          <box size="0.080 0.300 0.510" />
+        </geometry>
+        <material name="Blue" />
+      </visual>
+      <collision>
+        <origin xyz="0 0 0.255" rpy="0 0 0" />
+        <geometry>
+          <box size="0.080 0.300 0.510" />
+        </geometry>
+        <material name="Blue" />
+      </collision>
     </link>
     <joint name="base_footprint_joint" type="fixed">
@@ -133,4 +155,9 @@
       <child link="base_link" />
     </joint>
+    <joint name="vertical_body_joint" type="fixed">
+      <origin xyz="0 0 0.105" rpy="0 0 0" />
+      <parent link="base_footprint" />
+      <child link="vertical_body" />
+    </joint>
     <joint name="base_wall_sensor_joint" type="fixed">
       <origin xyz="0.09 -0.120 0.042" rpy="0 0 -1.0" />
@@ -169,5 +196,5 @@
     </joint>
     <joint name="cam_pan_joint" type="revolute">
-      <origin xyz="0.0 0.0 0.565" rpy="0 0 0" />
+      <origin xyz="0.0 0.0 0.630" rpy="0 0 0" />
       <axis xyz="0 0 1"/>
       <limit upper="1.57" lower="-1.57" effort="10" velocity="10"/>
@@ -183,5 +210,5 @@
     </link>
     <joint name="cam_tilt_joint" type="revolute">
-      <origin xyz="0.0 0.0 0.060" rpy="0 0 0" />
+      <origin xyz="0.0 0.0 0.053" rpy="0 0 0" />
       <axis xyz="0 1 0"/>
       <limit upper="1.57" lower="-1.57" effort="10" velocity="10"/>
@@ -197,5 +224,5 @@
     </link>
     <joint name="oakd_base" type="fixed">
-      <origin xyz="0.095 0 0.028" rpy="0 0 0" />
+      <origin xyz="0.105 0 0.045" rpy="0 0 0" />
       <parent link="cam_tilt_to_oakd_base" />
       <child link="oakd" />
@@ -203,30 +230,4 @@
     <xacro:create_wheel prefix="left" y_offset="${wheel_separation / 2}" wheel_radius="${wheel_radius}" wheel_width="${wheel_width}"/>
     <xacro:create_wheel prefix="right" y_offset="${wheel_separation / -2}" wheel_radius="${wheel_radius}" wheel_width="${wheel_width}"/>
-    <!--<link name="rear_wheel_link">
-    <inertial>
-      <origin xyz="0 0 0"/>
-      <mass value="0.001" />
-      <inertia ixx="0.0001" ixy="0.0" ixz="0.0"
-        iyy="0.0001" iyz="0.0" izz="0.0001" />
-    </inertial>
-    <visual>
-      <origin xyz="0 0 0" rpy="0 ${PI/2} ${PI/2}"/>
-      <geometry>
-        <sphere radius="0.015" />
-      </geometry>
-    </visual>
-    <collision>
-      <origin xyz="0 0 0" rpy="0 ${PI/2} ${PI/2}" />
-      <geometry>
-        <sphere radius="0.015" />
-      </geometry>
-    </collision>
-    </link>
-    <joint name="rear_castor_joint" type="fixed">
-      <origin xyz="-0.13 0 0.0" rpy="0 0 0"/>
-      <parent link="base_link"/>
-      <child link="rear_wheel_link"/>
-      <axis xyz="0 1 0"/>
-    </joint>-->
     <link name="front_wheel_link">
     <inertial>

Commit message: Support 3-finger end effector

File: create_description/urdf/create_2.urdf.xacro (robot description, xacro)
@@ -8,4 +8,6 @@
   </xacro:create_base>
   <xacro:property name="PI" value="3.1415926535897931" />
+  <!--xacro:property name="eef" value="eef_2_finger"/-->
+  <xacro:property name="eef" value="eef_3_finger"/>
   <joint name="xarm_base_joint" type="fixed">
         <parent link="base_footprint"/>
